File: designs-kicad/WifiSensor/WifiSensorArrayShield.kicad_pcb (KiCad board)
At the start: 2 copper layers, 7 parts, among them P1 PIR Sensor, P2 Light Sensor, P3 Sound Sensor, U1 ESP-12E

Commit message: no message
Routing:
- net Net-(P1-Pad2): track 20.1 -> 0.00 mm
